Commit message: Added gripper, could be better

File: poke_description/urdf/poke.xacro (robot description, xacro)
@@ -10,4 +10,12 @@
   <xacro:property name="l2" value="0.1" />         <!-- Cylinder Length Secondary-->
   <xacro:property name="mass" value="1e-2" />       <!-- arbitrary value for mass -->
+  <xacro:property name="radius_5" value="0.025" /><!--gripper base redius/width-->
+  <xacro:property name="radius_6" value="0.02" /> <!--finger radius/length-->
+  <xacro:property name="length_5" value="0.15" /> <!--gripper base length-->
+  <xacro:property name="length_6" value="0.07" /> <!--finger length-->
+   <xacro:property name="radius_52" value="0.025" /><!--gripper base redius/width-->
+   <xacro:property name="radius_62" value="0.02" /> <!--finger radius/length-->
+   <xacro:property name="length_62" value="0.07" /> <!--finger length-->
+   <xacro:property name="mass_62" value="0.2" />
   <xacro:property name="cam_name" value="cameraB"/>
   <!-- Imports -->
@@ -58,7 +66,10 @@
   <!-- Wrist [p3] -->
   <cSeg parent="p2_link" name="p3" color="green"/>
-  <!-- Camera -->
+  <!--gripper-->
+  <gripper parent="p3_link" name="gripper"/>
+  <!-- Camera
   <cam parent="p3_link" name="${cam_name}" />
   <cam_gazebo camName="${cam_name}" />
+-->
   <!-- Motor Transmission -->
   <mtrT jointName="p0_joint"/>
@@ -66,4 +77,6 @@
   <mtrT jointName="p2_joint"/>
   <mtrT jointName="p3_joint"/>
+  <mtrT jointName="gripper_1"/>
+  <mtrT jointName="gripper_2"/>
   </xacro:macro>
 </robot>

File: poke_description/urdf/poke_hardware.xacro (robot description, xacro)
@@ -1,4 +1,14 @@
 <?xml version="1.0" encoding="UTF-8"?>
 <robot xmlns:xacro="http://ros.org/wiki/xacro">
+    <xacro:macro name="inertial_block" params="mass length radius">
+        <inertial>
+        <origin xyz="0 0 ${length/2}" rpy="0 0 0"/>
+        <mass value="${mass}"/>
+        <inertia
+            ixx="${mass / 12.0 * (2*radius*2*radius + length*length)}" ixy="0.0" ixz="0.0"
+            iyy="${mass / 12.0 * (length*length + 2*radius*2*radius)}" iyz="0.0"
+            izz="${mass / 12.0 * (2*radius*2*radius + 2*radius*2*radius)}" />
+    </inertial>
+    </xacro:macro>
    <!-- macro for arm base mount -->
    <xacro:macro name="base_mount" params="parent name color *origin">
@@ -150,4 +160,74 @@
          </collision>
       </link>
+   </xacro:macro>
+   <xacro:macro name="gripper" params="parent name">
+      <joint name ="gripper_1" type="prismatic">
+         <origin xyz="0.0 0.0 ${radius_5 + length_6/2.0}" rpy="0.0 0.0 0.0"/>
+         <axis xyz="0 0 0"/>
+         <parent link="${parent}" />
+         <child link="gripper_link_1"/>
+         <limit lower="${radius_62/2.0}" upper="0.05" effort="100.0" velocity="1.0"/>
+      </joint>
+      <joint name ="gripper_2" type="prismatic">
+        <origin xyz="0.0 0.0 ${radius_5 + length_6/2.0}" rpy="0.0 0.0 0.0"/>
+        <parent link="${parent}" />
+        <child link="gripper_link_2"/>
+        <axis xyz="0.0 0.0 0.0"/>
+        <limit lower="-0.05" upper="${-radius_6/2.0}" effort="100.0" velocity="1.0"/>
+      </joint>
+     <joint name="gripper_frame_joint" type="fixed">
+        <origin xyz="0.0 0.0 ${radius_52*2 + length_62/2 + 0.01}" rpy="0.0 0.0 0.0"/>
+        <parent link="${parent}"/>
+        <child link="gripper_frame_cp"/>
+        <axis xyz="0.0 0.0 0.0"/>
+    </joint>
+     <link name="gripper_link_1">
+        <xacro:inertial_block mass="${mass_62}" length="${length_62}" radius="${radius_62}"/>
+        <visual>
+            <origin xyz="0.0 0.0 ${radius_62/2.0}" rpy="0.0 0.0 0.0"/>
+            <geometry>
+                <box size="${radius_62} ${radius_62*2} ${length_62}"/>
+            </geometry>
+            <material name="Grey"/>
+        </visual>
+        <collision>
+            <origin xyz="0.0 0.0 ${radius_62/2.0}" rpy="0.0 0.0 0.0"/>
+            <geometry>
+                <box size="${radius_62*2} ${radius_62*2} ${length_62}"/>
+            </geometry>
+        </collision>
+    </link>
+     <link name="gripper_link_2">
+        <xacro:inertial_block mass="${mass_62}" length="${length_62}" radius="${radius_62}"/>
+        <visual>
+            <origin xyz="0.0 0.0 ${radius_62/2.0}" rpy="0.0 0.0 0.0"/>
+            <geometry>
+                <box size="${radius_62} ${radius_62*2} ${length_62}"/>
+            </geometry>
+            <material name="Grey"/>
+        </visual>
+        <collision>
+            <origin xyz="0.0 0.0 ${radius_62/2.0}" rpy="0.0 0.0 0.0"/>
+            <geometry>
+                <box size="${radius_62*2} ${radius_62*2} ${length_62}"/>
+            </geometry>
+        </collision>
+    </link>
+    <link name="gripper_frame_cp">
+        <xacro:inertial_block mass="${0.001}" length="${0.001}" radius="${0.001}"/>
+        <visual>
+            <origin xyz="0.0 0.0 0.0" rpy="0.0 0.0 0.0"/>
+            <geometry>
+                <box size="${0.001} ${0.001} ${0.001}"/>
+            </geometry>
+            <material name="Grey"/>
+        </visual>
+        <collision>
+            <origin xyz="0.0 0.0 0.0" rpy="0.0 0.0 0.0"/>
+            <geometry>
+                <box size="${0.001} ${0.001} ${0.001}"/>
+            </geometry>
+        </collision>
+    </link>
    </xacro:macro>
    <xacro:macro name="cam" params="parent name">

Commit message: Working Gripper, almost ready

File: poke_description/urdf/poke.xacro (robot description, xacro)
@@ -16,5 +16,5 @@
    <xacro:property name="radius_52" value="0.025" /><!--gripper base redius/width-->
    <xacro:property name="radius_62" value="0.02" /> <!--finger radius/length-->
-   <xacro:property name="length_62" value="0.07" /> <!--finger length-->
+   <xacro:property name="length_62" value="0.1" /> <!--finger length-->
    <xacro:property name="mass_62" value="0.2" />
   <xacro:property name="cam_name" value="cameraB"/>

File: poke_description/urdf/poke_hardware.xacro (robot description, xacro)
@@ -163,19 +163,20 @@
    <xacro:macro name="gripper" params="parent name">
       <joint name ="gripper_1" type="prismatic">
-         <origin xyz="0.0 0.0 ${radius_5 + length_6/2.0}" rpy="0.0 0.0 0.0"/>
+         <origin xyz="0.0 0.0 ${radius_52 + length_62/2.0}" rpy="0.0 0.0 0.0"/>
          <axis xyz="0 0 0"/>
          <parent link="${parent}" />
          <child link="gripper_link_1"/>
-         <limit lower="${radius_62/2.0}" upper="0.05" effort="100.0" velocity="1.0"/>
+         <limit lower="${radius_62/2.0}" upper="0.5" effort="100.0" velocity="1.0"/>
       </joint>
       <joint name ="gripper_2" type="prismatic">
-        <origin xyz="0.0 0.0 ${radius_5 + length_6/2.0}" rpy="0.0 0.0 0.0"/>
+        <origin xyz="0.0 0.0 ${radius_52 + length_62/2.0}" rpy="0.0 0.0 0.0"/>
         <parent link="${parent}" />
         <child link="gripper_link_2"/>
         <axis xyz="0.0 0.0 0.0"/>
-        <limit lower="-0.05" upper="${-radius_6/2.0}" effort="100.0" velocity="1.0"/>
+        <limit lower="-0.5" upper="${-radius_62/2.0}" effort="25.0" velocity="1.0"/>
       </joint>
      <joint name="gripper_frame_joint" type="fixed">
-        <origin xyz="0.0 0.0 ${radius_52*2 + length_62/2 + 0.01}" rpy="0.0 0.0 0.0"/>
+        <!--origin xyz="0.0 0.0 ${radius_52*2 + length_62/2 + 0.01}" rpy="0.0 0.0 0.0"/-->
+        <origin xyz="0.0 0.0 0.0" rpy="0.0 0.0 0.0"/>
         <parent link="${parent}"/>
         <child link="gripper_frame_cp"/>
@@ -219,5 +220,5 @@
             <origin xyz="0.0 0.0 0.0" rpy="0.0 0.0 0.0"/>
             <geometry>
-                <box size="${0.001} ${0.001} ${0.001}"/>
+                <box size="${0.1} ${0.05} ${0.05}"/>
             </geometry>
             <material name="Grey"/>
@@ -226,5 +227,5 @@
             <origin xyz="0.0 0.0 0.0" rpy="0.0 0.0 0.0"/>
             <geometry>
-                <box size="${0.001} ${0.001} ${0.001}"/>
+                <box size="${0.1} ${0.05} ${0.05}"/>
             </geometry>
         </collision>

Commit message: Changes to boti

File: poke_description/urdf/poke.xacro (robot description, xacro)
@@ -15,6 +15,6 @@
   <xacro:property name="length_6" value="0.07" /> <!--finger length-->
    <xacro:property name="radius_52" value="0.025" /><!--gripper base redius/width-->
-   <xacro:property name="radius_62" value="0.02" /> <!--finger radius/length-->
-   <xacro:property name="length_62" value="0.1" /> <!--finger length-->
+   <xacro:property name="radius_62" value="0.05" /> <!--finger radius/length-->
+   <xacro:property name="length_62" value="0.15" /> <!--finger length-->
    <xacro:property name="mass_62" value="0.2" />
   <xacro:property name="cam_name" value="cameraB"/>

File: poke_description/urdf/poke1.urdf (robot description, URDF)
Before this commit: robot poke_arm_main, 10 links, 9 joints
Links:
- link gripper_link_1: mass 0.2 -> 0.02
- link gripper_link_2: mass 0.2 -> 0.02
Joints:
- joint gripper_1: limit lower=0.025 upper=0.5 effort=30.0 velocity=1.0 -> lower=0.025 upper=0.5 effort=10.0 velocity=1.0
- joint gripper_2: limit lower=-0.5 upper=-0.025 effort=30.0 velocity=1.0 -> lower=-0.5 upper=-0.025 effort=10.0 velocity=1.0

File: poke_description/urdf/poke_hardware.xacro (robot description, xacro)
@@ -46,5 +46,5 @@
          <child link="${name}_link" />
          <axis xyz="0 1 0" />
-         <limit lower="${llimit}" upper="${ulimit}" velocity="${vlimit}" effort="30" />
+         <limit lower="${llimit}" upper="${ulimit}" velocity="${vlimit}" effort="100" />
          <!--origin rpy="0 0 0" xyz="0.0 0.0 ${l1+jr}" /-->
       </joint>
@@ -92,5 +92,5 @@
          <child link="${name}_link" />
          <axis xyz="0 1 0" />
-         <limit lower="${llimit}" upper="${ulimit}" velocity="${vlimit}" effort="30" />
+         <limit lower="${llimit}" upper="${ulimit}" velocity="${vlimit}" effort="100" />
          <origin rpy="0 0 0" xyz="0.0 0.0 ${l1+jr}" />
       </joint>
@@ -167,5 +167,5 @@
          <parent link="${parent}" />
          <child link="gripper_link_1"/>
-         <limit lower="${radius_62/2.0}" upper="0.5" effort="100.0" velocity="1.0"/>
+         <limit lower="${radius_62/2.0}" upper="0.5" effort="30.0" velocity="1.0"/>
       </joint>
       <joint name ="gripper_2" type="prismatic">
@@ -174,5 +174,5 @@
         <child link="gripper_link_2"/>
         <axis xyz="0.0 0.0 0.0"/>
-        <limit lower="-0.5" upper="${-radius_62/2.0}" effort="25.0" velocity="1.0"/>
+        <limit lower="-0.5" upper="${-radius_62/2.0}" effort="30.0" velocity="1.0"/>
       </joint>
      <joint name="gripper_frame_joint" type="fixed">
@@ -188,13 +188,21 @@
             <origin xyz="0.0 0.0 ${radius_62/2.0}" rpy="0.0 0.0 0.0"/>
             <geometry>
-                <box size="${radius_62} ${radius_62*2} ${length_62}"/>
+                <box size="${radius_62/2} ${radius_62*2} ${length_62}"/>
             </geometry>
             <material name="Grey"/>
         </visual>
-        <collision>
+        <collision name="gripper_touch_1">
             <origin xyz="0.0 0.0 ${radius_62/2.0}" rpy="0.0 0.0 0.0"/>
             <geometry>
-                <box size="${radius_62*2} ${radius_62*2} ${length_62}"/>
-            </geometry>
+                <box size="${radius_62/2} ${radius_62*2} ${length_62}"/>
+            </geometry>
+            <surface>
+               <friction>
+                  <ode>
+                  <slip1>1.0</slip1>
+                  <slip2>1.0</slip2>
+                  </ode>
+               </friction>
+            </surface>
         </collision>
     </link>
@@ -204,13 +212,27 @@
             <origin xyz="0.0 0.0 ${radius_62/2.0}" rpy="0.0 0.0 0.0"/>
             <geometry>
-                <box size="${radius_62} ${radius_62*2} ${length_62}"/>
+                <box size="${radius_62/2} ${radius_62*2} ${length_62}"/>
             </geometry>
             <material name="Grey"/>
         </visual>
-        <collision>
+        <collision name="gripper_touch_2">
             <origin xyz="0.0 0.0 ${radius_62/2.0}" rpy="0.0 0.0 0.0"/>
             <geometry>
-                <box size="${radius_62*2} ${radius_62*2} ${length_62}"/>
-            </geometry>
+                <box size="${radius_62/2} ${radius_62*2} ${length_62}"/>
+            </geometry>
+            <surface>
+               <contact>
+                  <ode>
+                     <min_depth>0.003</min_depth>
+                     <max_vel>0.0</max_vel>
+                  </ode>
+               </contact>
+               <friction>
+                  <ode>
+                     <mu>10.0</mu>
+                     <mu2>10.0</mu2>
+                  </ode>
+               </friction>
+            </surface>
         </collision>
     </link>
