Commit message: Moveit and owot working

File: poke_description/urdf/poke.urdf (robot description, URDF)
Before this commit: robot poke_arm_main, 10 links, 9 joints
Links:
- link gripper_frame_cp: mass 0.001 -> 0.01; geometry collision box size=0.0225 0.03375 0.045; visual box size=0.0225 0.03375 0.045
Joints:
- joint gripper_1: axis 0 0 0 -> 1 0 0
- joint gripper_2: axis 0.0 0.0 0.0 -> 1 0 0
- joint gripper_frame_joint: axis 0.0 0.0 0.0 -> 0 0 0; origin xyz=0.0 0.0 0.0 rpy=0.0 0.0 0.0 -> xyz=0 0 0.036 rpy=0 -1.570795 0
- joint p0_joint: limit lower=-1.04719666667 upper=1.5079632 effort=100 velocity=5 -> lower=-3.14159 upper=3.14159 effort=100 velocity=5
- joint p1_joint: limit lower=0 upper=2.09439333333 effort=100 velocity=5 -> lower=-3.14159 upper=3.14159 effort=100 velocity=5
- joint p2_joint: limit lower=-2.09439333333 upper=2.09439333333 effort=100 velocity=5 -> lower=-3.14159 upper=3.14159 effort=100 velocity=5

File: poke_description/urdf/poke.xacro (robot description, xacro)
@@ -14,8 +14,8 @@
   <xacro:property name="length_5" value="0.15" /> <!--gripper base length-->
   <xacro:property name="length_6" value="0.07" /> <!--finger length-->
-   <xacro:property name="radius_52" value="0.025" /><!--gripper base redius/width-->
-   <xacro:property name="radius_62" value="0.05" /> <!--finger radius/length-->
-   <xacro:property name="length_62" value="0.15" /> <!--finger length-->
-   <xacro:property name="mass_62" value="0.2" />
+  <xacro:property name="radius_52" value="0.025" /><!--gripper base redius/width-->
+  <xacro:property name="radius_62" value="0.05" /> <!--finger radius/length-->
+  <xacro:property name="length_62" value="0.15" /> <!--finger length-->
+  <xacro:property name="mass_62" value="0.2" />
   <xacro:property name="cam_name" value="cameraB"/>
   <!-- Imports -->
@@ -53,15 +53,15 @@
   <!-- Torso [p0] -->
   <segmentL parent="baseMount_link" name="p0" color="orange"
-    llimit="-${1/3*PI}" ulimit="${0.48*PI}" vlimit="5">
+    llimit="-${PI}" ulimit="${PI}" vlimit="5">
     <origin rpy="0 0 0" xyz="0.0 0.0 ${l0+jr}" />
   </segmentL>
   <!-- Shoulder [p1] -->
   <segmentL parent="p0_link" name="p1" color="orange"
-    llimit="0" ulimit="${2/3*PI}" vlimit="5">
+    llimit="-${PI}" ulimit="${PI}" vlimit="5">
     <origin rpy="0 0 0" xyz="0.0 0.0 ${l1+jr}" />
   </segmentL>
   <!-- Arm [p2] -->
   <segmentS parent="p1_link" name="p2" color="orange"
-    llimit="-${2/3*PI}" ulimit="${2/3*PI}" vlimit="5"/>
+    llimit="-${PI}" ulimit="${PI}" vlimit="5"/>
   <!-- Wrist [p3] -->
   <cSeg parent="p2_link" name="p3" color="green"/>

File: poke_description/urdf/poke1.urdf (robot description, URDF)
Before this commit: robot poke_arm_main, 10 links, 9 joints
Links:
- link gripper_frame_cp: mass 0.001 -> 0.01

File: poke_description/urdf/poke_hardware.xacro (robot description, xacro)
@@ -164,5 +164,5 @@
       <joint name ="gripper_1" type="prismatic">
          <origin xyz="0.0 0.0 ${radius_52 + length_62/2.0}" rpy="0.0 0.0 0.0"/>
-         <axis xyz="0 0 0"/>
+         <axis xyz="1 0 0"/>
          <parent link="${parent}" />
          <child link="gripper_link_1"/>
@@ -173,36 +173,28 @@
         <parent link="${parent}" />
         <child link="gripper_link_2"/>
-        <axis xyz="0.0 0.0 0.0"/>
+        <axis xyz="1 0 0"/>
         <limit lower="-0.5" upper="${-radius_62/2.0}" effort="30.0" velocity="1.0"/>
       </joint>
      <joint name="gripper_frame_joint" type="fixed">
         <!--origin xyz="0.0 0.0 ${radius_52*2 + length_62/2 + 0.01}" rpy="0.0 0.0 0.0"/-->
-        <origin xyz="0.0 0.0 0.0" rpy="0.0 0.0 0.0"/>
+        <axis xyz="0 0 0" />
+         <!-- Use the joint to orientate the camera -->
+         <origin xyz="0 0 ${.8*jr}" rpy="0 ${-PI/2} 0" />
         <parent link="${parent}"/>
         <child link="gripper_frame_cp"/>
-        <axis xyz="0.0 0.0 0.0"/>
     </joint>
      <link name="gripper_link_1">
         <xacro:inertial_block mass="${mass_62}" length="${length_62}" radius="${radius_62}"/>
         <visual>
-            <origin xyz="0.0 0.0 ${radius_62/2.0}" rpy="0.0 0.0 0.0"/>
+            <origin xyz="${radius_62/2} 0.0 ${radius_62/2.0}" rpy="0.0 0.0 0.0"/>
             <geometry>
                 <box size="${radius_62/2} ${radius_62*2} ${length_62}"/>
             </geometry>
-            <material name="Grey"/>
         </visual>
-        <collision name="gripper_touch_1">
-            <origin xyz="0.0 0.0 ${radius_62/2.0}" rpy="0.0 0.0 0.0"/>
+        <collision>
+            <origin xyz="${radius_62/2} 0.0 ${radius_62/2.0}" rpy="0.0 0.0 0.0"/>
             <geometry>
                 <box size="${radius_62/2} ${radius_62*2} ${length_62}"/>
             </geometry>
-            <surface>
-               <friction>
-                  <ode>
-                  <slip1>1.0</slip1>
-                  <slip2>1.0</slip2>
-                  </ode>
-               </friction>
-            </surface>
         </collision>
     </link>
@@ -210,47 +202,38 @@
         <xacro:inertial_block mass="${mass_62}" length="${length_62}" radius="${radius_62}"/>
         <visual>
-            <origin xyz="0.0 0.0 ${radius_62/2.0}" rpy="0.0 0.0 0.0"/>
+            <origin xyz="${-radius_62/2} 0.0 ${radius_62/2.0}" rpy="0.0 0.0 0.0"/>
             <geometry>
                 <box size="${radius_62/2} ${radius_62*2} ${length_62}"/>
             </geometry>
-            <material name="Grey"/>
         </visual>
-        <collision name="gripper_touch_2">
-            <origin xyz="0.0 0.0 ${radius_62/2.0}" rpy="0.0 0.0 0.0"/>
+        <collision>
+            <origin xyz="{-radius_62/2} 0.0 ${radius_62/2.0}" rpy="0.0 0.0 0.0"/>
             <geometry>
                 <box size="${radius_62/2} ${radius_62*2} ${length_62}"/>
             </geometry>
-            <surface>
-               <contact>
-                  <ode>
-                     <min_depth>0.003</min_depth>
-                     <max_vel>0.0</max_vel>
-                  </ode>
-               </contact>
-               <friction>
-                  <ode>
-                     <mu>10.0</mu>
-                     <mu2>10.0</mu2>
-                  </ode>
-               </friction>
-            </surface>
         </collision>
     </link>
     <link name="gripper_frame_cp">
-        <xacro:inertial_block mass="${0.001}" length="${0.001}" radius="${0.001}"/>
         <visual>
-            <origin xyz="0.0 0.0 0.0" rpy="0.0 0.0 0.0"/>
-            <geometry>
-                <box size="${0.1} ${0.05} ${0.05}"/>
-            </geometry>
-            <material name="Grey"/>
-        </visual>
-        <collision>
-            <origin xyz="0.0 0.0 0.0" rpy="0.0 0.0 0.0"/>
-            <geometry>
-                <box size="${0.1} ${0.05} ${0.05}"/>
-            </geometry>
-        </collision>
-    </link>
+            <origin xyz="0 0 0" rpy="0 0 0" />
+            <geometry>
+               <box size="${jr/2} ${.75*jr} ${jr}" />
+            </geometry>
+            <material name="grey">
+               <color rgba="0.2 0.2 0.2 1.0" />
+            </material>
+         </visual>
+         <collision>
+            <origin xyz="0 0 0" rpy="0 0 0" />
+            <geometry>
+               <box size="${jr/2} ${.75*jr} ${jr}" />
+            </geometry>
+         </collision>
+         <inertial>
+            <mass value="0.01" />
+            <origin xyz="0 0 0" rpy="0 0 0" />
+            <inertia ixx="1e-6" ixy="0" ixz="0" iyy="1e-6" iyz="0" izz="1e-6" />
+         </inertial>
+      </link>
    </xacro:macro>
    <xacro:macro name="cam" params="parent name">

Commit message: What a piece of junk, ya jala todo mi wobot :) <3

File: poke_description/urdf/poke.urdf (robot description, URDF)
Before this commit: robot poke_arm_main, 10 links, 9 joints
Joints:
- joint p0_joint: limit lower=-3.14159 upper=3.14159 effort=100 velocity=5 -> lower=-1.5708 upper=1.5708 effort=100 velocity=5
